File: effectorboardtop_kicad.sch (KiCad schematic (older format))
At the start: 39 parts

Commit message: garbage removed
Parts:
- removed C?: CP1, ~, symbol CP1
- removed PWR? (x6): GND, symbol GND
- added U?: QFP64, MODULE, symbol QFP64
Connections:
- net labels added: GND
Changed lines of the file:
@@
 LIBS:contrib
 LIBS:valves
+LIBS:effectorboardtop_kicad-cache
 EELAYER 27 0
 EELAYER END
@@
 Sheet 1 1
 Title ""
-Date "8 oct 2015"
+Date "9 oct 2015"
 Rev ""
 Comp ""
@@
 $EndDescr
 $Comp
-L GND PWR?
+L GND #PWR01
 U 1 1 4E44605E
 P 12800 9050
-F 0 "" H 12800 9050 60  0001 C CNN
+F 0 "#PWR01" H 12850 9100 60  0001 C CNN
 F 1 "GND" H 12800 8980 30  0000 C CNN
 F 2 "" H 12800 9050 60  0001 C CNN
@@
 $EndComp
 $Comp
-L GND PWR?
+L GND #PWR02
 U 1 1 4E44605E
 P 7900 10150
-F 0 "" H 7900 10150 60  0001 C CNN
+F 0 "#PWR02" H 7950 10200 60  0001 C CNN
 F 1 "GND" H 7900 10080 30  0000 C CNN
 F 2 "" H 7900 10150 60  0001 C CNN
@@
 $EndComp
 $Comp
-L GND PWR?
+L GND #PWR03
 U 1 1 4E44605E
 P 7900 4250
-F 0 "" H 7900 4250 60  0001 C CNN
+F 0 "#PWR03" H 7950 4300 60  0001 C CNN
 F 1 "GND" H 7900 4180 30  0000 C CNN
 F 2 "" H 7900 4250 60  0001 C CNN
@@
 $EndComp
 $Comp
-L GND PWR?
+L GND #PWR04
 U 1 1 4E44605E
 P 2600 3650
-F 0 "" H 2600 3650 60  0001 C CNN
+F 0 "#PWR04" H 2650 3700 60  0001 C CNN
 F 1 "GND" H 2600 3580 30  0000 C CNN
 F 2 "" H 2600 3650 60  0001 C CNN
@@
 $EndComp
 $Comp
-L GND PWR?
+L GND #PWR05
 U 1 1 4E44605E
 P 12900 2650
-F 0 "" H 12900 2650 60  0001 C CNN
+F 0 "#PWR05" H 12950 2700 60  0001 C CNN
 F 1 "GND" H 12900 2580 30  0000 C CNN
 F 2 "" H 12900 2650 60  0001 C CNN
@@
 $EndComp
 $Comp
-L GND PWR?
+L GND #PWR06
 U 1 1 4E44605E
 P 14300 6050
-F 0 "" H 14300 6050 60  0001 C CNN
+F 0 "#PWR06" H 14350 6100 60  0001 C CNN
 F 1 "GND" H 14300 5980 30  0000 C CNN
 F 2 "" H 14300 6050 60  0001 C CNN
@@
 $Comp
 L CP1 C?
-U 1 1 561665BF
-P 13100 3550
-F 0 "C?" H 13150 3650 50  0000 L CNN
-F 1 "CP1" H 13150 3450 50  0000 L CNN
-F 2 "~" H 13100 3550 60  0000 C CNN
-F 3 "~" H 13100 3550 60  0000 C CNN
-	1    13100 3550
-	1    0    0    -1
-$EndComp
-$Comp
-L CP1 C?
 U 1 1 561665DD
 P 8300 8250
@@
 	1    0    0    -1
 $EndComp
+$Comp
+L QFP64 U?
+U 1 1 56166E26
+P -350 9250
+F 0 "U?" H -350 9150 50  0000 C CNN
+F 1 "QFP64" H -350 9350 50  0000 C CNN
+F 2 "MODULE" H -350 9250 50  0001 C CNN
+F 3 "DOCUMENTATION" H -350 9250 50  0001 C CNN
+	1    -350 9250
+	1    0    0    -1
+$EndComp

Commit message: old symbols replaced manually
Parts:
- removed U?: QFP64, MODULE, symbol QFP64
- added PWR? (x6): GND, symbol GND
Connections:
- net labels removed: GND

Commit message: first ERC performed
Parts:
- removed PWR? (x6): GND, symbol GND
- gave numbers to parts that had none: 32
Connections:
- net labels added: GND
Changed lines of the file:
@@
 $EndDescr
 $Comp
-L GND PWR?
-U 1 1 4E44605E
+L GND #PWR01
+U 1 1 5617B4B1
 P 12800 9050
-F 0 "" H 12800 9050 60  0001 C CNN
+F 0 "#PWR01" H 12850 9100 60  0001 C CNN
 F 1 "GND" H 12800 8980 30  0000 C CNN
 F 2 "" H 12800 9050 60  0001 C CNN
@@
 $EndComp
 $Comp
-L GND PWR?
-U 1 1 4E44605E
+L GND #PWR02
+U 1 1 5617B4B2
 P 7900 10150
-F 0 "" H 7900 10150 60  0001 C CNN
+F 0 "#PWR02" H 7950 10200 60  0001 C CNN
 F 1 "GND" H 7900 10080 30  0000 C CNN
 F 2 "" H 7900 10150 60  0001 C CNN
@@
 $EndComp
 $Comp
-L GND PWR?
-U 1 1 4E44605E
+L GND #PWR03
+U 1 1 5617B4B3
 P 7900 4250
-F 0 "" H 7900 4250 60  0001 C CNN
+F 0 "#PWR03" H 7950 4300 60  0001 C CNN
 F 1 "GND" H 7900 4180 30  0000 C CNN
 F 2 "" H 7900 4250 60  0001 C CNN
@@
 $EndComp
 $Comp
-L GND PWR?
-U 1 1 4E44605E
+L GND #PWR04
+U 1 1 5617B4B4
 P 2600 3650
-F 0 "" H 2600 3650 60  0001 C CNN
+F 0 "#PWR04" H 2650 3700 60  0001 C CNN
 F 1 "GND" H 2600 3580 30  0000 C CNN
 F 2 "" H 2600 3650 60  0001 C CNN
@@
 $EndComp
 $Comp
-L GND PWR?
-U 1 1 4E44605E
+L GND #PWR05
+U 1 1 5617B4B5
 P 12900 2650
-F 0 "" H 12900 2650 60  0001 C CNN
+F 0 "#PWR05" H 12950 2700 60  0001 C CNN
 F 1 "GND" H 12900 2580 30  0000 C CNN
 F 2 "" H 12900 2650 60  0001 C CNN
@@
 $EndComp
 $Comp
-L GND PWR?
-U 1 1 4E44605E
-P 14300 6050
-F 0 "" H 14300 6050 60  0001 C CNN
-F 1 "GND" H 14300 5980 30  0000 C CNN
-F 2 "" H 14300 6050 60  0001 C CNN
-F 3 "" H 14300 6050 60  0001 C CNN
-	1    14300 6050
-	1    0    0    -1
-$EndComp
-$Comp
-L R R?
+L R R2
 U 1 1 56160318
 P 4800 2400
-F 0 "R?" V 4880 2400 40  0000 C CNN
+F 0 "R2" V 4880 2400 40  0000 C CNN
 F 1 "47k" V 4807 2401 40  0000 C CNN
 F 2 "~" V 4730 2400 30  0000 C CNN
@@
 $EndComp
 $Comp
-L R R?
+L R R1
 U 1 1 5616246B
 P 4300 2900
-F 0 "R?" V 4380 2900 40  0000 C CNN
+F 0 "R1" V 4380 2900 40  0000 C CNN
 F 1 "47k" V 4307 2901 40  0000 C CNN
 F 2 "~" V 4230 2900 30  0000 C CNN
@@
 $EndComp
 $Comp
-L R R?
+L R R3
 U 1 1 56162487
 P 5300 2900
-F 0 "R?" V 5380 2900 40  0000 C CNN
+F 0 "R3" V 5380 2900 40  0000 C CNN
 F 1 "47k" V 5307 2901 40  0000 C CNN
 F 2 "~" V 5230 2900 30  0000 C CNN
@@
 $EndComp
 $Comp
-L R R?
+L R R4
 U 1 1 56162491
 P 5900 2400
-F 0 "R?" V 5980 2400 40  0000 C CNN
+F 0 "R4" V 5980 2400 40  0000 C CNN
 F 1 "47k" V 5907 2401 40  0000 C CNN
 F 2 "~" V 5830 2400 30  0000 C CNN
@@
 $EndComp
 $Comp
-L R R?
+L R R5
 U 1 1 56162497
 P 6400 2900
-F 0 "R?" V 6480 2900 40  0000 C CNN
+F 0 "R5" V 6480 2900 40  0000 C CNN
 F 1 "47k" V 6407 2901 40  0000 C CNN
 F 2 "~" V 6330 2900 30  0000 C CNN
@@
 $EndComp
 $Comp
-L R R?
+L R R6
 U 1 1 5616249D
 P 6900 2400
-F 0 "R?" V 6980 2400 40  0000 C CNN
+F 0 "R6" V 6980 2400 40  0000 C CNN
 F 1 "47k" V 6907 2401 40  0000 C CNN
 F 2 "~" V 6830 2400 30  0000 C CNN
@@
 $EndComp
 $Comp
-L R R?
+L R R13
 U 1 1 561624ED
 P 12050 6150
-F 0 "R?" V 12130 6150 40  0000 C CNN
+F 0 "R13" V 12130 6150 40  0000 C CNN
 F 1 "10k" V 12057 6151 40  0000 C CNN
 F 2 "~" V 11980 6150 30  0000 C CNN
@@
 $EndComp
 $Comp
-L R R?
+L R R14
 U 1 1 56162507
 P 12050 6750
-F 0 "R?" V 12130 6750 40  0000 C CNN
+F 0 "R14" V 12130 6750 40  0000 C CNN
 F 1 "20k" V 12057 6751 40  0000 C CNN
 F 2 "~" V 11980 6750 30  0000 C CNN
@@
 $EndComp
 $Comp
-L R R?
+L R R12
 U 1 1 56162522
 P 11950 8750
-F 0 "R?" V 12030 8750 40  0000 C CNN
+F 0 "R12" V 12030 8750 40  0000 C CNN
 F 1 "47k" V 11957 8751 40  0000 C CNN
 F 2 "~" V 11880 8750 30  0000 C CNN
@@
 $EndComp
 $Comp
-L R R?
+L R R10
 U 1 1 5616256E
 P 10950 5550
-F 0 "R?" V 11030 5550 40  0000 C CNN
+F 0 "R10" V 11030 5550 40  0000 C CNN
 F 1 "10k" V 10957 5551 40  0000 C CNN
 F 2 "~" V 10880 5550 30  0000 C CNN
@@
 $EndComp
 $Comp
-L R R?
+L R R8
 U 1 1 5616257D
 P 9150 5950
-F 0 "R?" V 9230 5950 40  0000 C CNN
+F 0 "R8" V 9230 5950 40  0000 C CNN
 F 1 "67k" V 9157 5951 40  0000 C CNN
 F 2 "~" V 9080 5950 30  0000 C CNN
@@
 $EndComp
 $Comp
-L R R?
+L R R7
 U 1 1 56162591
 P 8350 5950
-F 0 "R?" V 8430 5950 40  0000 C CNN
+F 0 "R7" V 8430 5950 40  0000 C CNN
 F 1 "67k" V 8357 5951 40  0000 C CNN
 F 2 "~" V 8280 5950 30  0000 C CNN
@@
 $EndComp
 $Comp
-L C C?
+L C C1
 U 1 1 561625BC
 P 7900 8250
-F 0 "C?" H 7900 8350 40  0000 L CNN
+F 0 "C1" H 7900 8350 40  0000 L CNN
 F 1 "0.1u" H 7906 8165 40  0000 L CNN
 F 2 "~" H 7938 8100 30  0000 C CNN
@@
 $EndComp
 $Comp
-L C C?
+L C C5
 U 1 1 561625EC
 P 9100 8250
-F 0 "C?" H 9100 8350 40  0000 L CNN
+F 0 "C5" H 9100 8350 40  0000 L CNN
 F 1 "0.1u" H 9106 8165 40  0000 L CNN
 F 2 "~" H 9138 8100 30  0000 C CNN
@@
 $EndComp
 $Comp
-L C C?
+L C C3
 U 1 1 561625F2
 P 8400 9550
-F 0 "C?" H 8400 9650 40  0000 L CNN
+F 0 "C3" H 8400 9650 40  0000 L CNN
 F 1 "0.1u" H 8406 9465 40  0000 L CNN
 F 2 "~" H 8438 9400 30  0000 C CNN
@@
 $EndComp
 $Comp
-L C C?
+L C C10
 U 1 1 5616264F
 P 12500 8750
-F 0 "C?" H 12500 8850 40  0000 L CNN
+F 0 "C10" H 12500 8850 40  0000 L CNN
 F 1 "0.1u" H 12506 8665 40  0000 L CNN
 F 2 "~" H 12538 8600 30  0000 C CNN
@@
 $EndComp
 $Comp
-L C C?
+L C C8
 U 1 1 56162673
 P 12100 7550
-F 0 "C?" H 12100 7650 40  0000 L CNN
+F 0 "C8" H 12100 7650 40  0000 L CNN
 F 1 "100p" H 12106 7465 40  0000 L CNN
 F 2 "~" H 12138 7400 30  0000 C CNN
@@
 $EndComp
 $Comp
-L R R?
+L R R15
 U 1 1 561626A0
 P 12550 8150
-F 0 "R?" V 12630 8150 40  0000 C CNN
+F 0 "R15" V 12630 8150 40  0000 C CNN
 F 1 "1" V 12557 8151 40  0000 C CNN
 F 2 "~" V 12480 8150 30  0000 C CNN
@@
 $EndComp
 $Comp
-L C C?
+L C C11
 U 1 1 561626B8
 P 12600 6150
-F 0 "C?" H 12600 6250 40  0000 L CNN
+F 0 "C11" H 12600 6250 40  0000 L CNN
 F 1 "0.47u" H 12606 6065 40  0000 L CNN
 F 2 "~" H 12638 6000 30  0000 C CNN
@@
 $EndComp
 $Comp
-L C C?
+L C C9
 U 1 1 561626DE
 P 12200 4550
-F 0 "C?" H 12200 4650 40  0000 L CNN
+F 0 "C9" H 12200 4650 40  0000 L CNN
 F 1 "0.047u" H 12206 4465 40  0000 L CNN
 F 2 "~" H 12238 4400 30  0000 C CNN
@@
 $EndComp
 $Comp
-L C C?
+L C C7
 U 1 1 561626F7
 P 10600 4950
-F 0 "C?" H 10600 5050 40  0000 L CNN
+F 0 "C7" H 10600 5050 40  0000 L CNN
 F 1 "47p" H 10606 4865 40  0000 L CNN
 F 2 "~" H 10638 4800 30  0000 C CNN
@@
 $EndComp
 $Comp
-L RVAR R?
+L RVAR R11
 U 1 1 56164440
 P 11950 8150
-F 0 "R?" V 12030 8100 50  0000 C CNN
+F 0 "R11" V 12030 8100 50  0000 C CNN
 F 1 "47k" V 11870 8210 50  0000 C CNN
 F 2 "~" H 11950 8150 60  0000 C CNN
@@
 $EndComp
 $Comp
-L RVAR R?
+L RVAR R9
 U 1 1 56165DDD
 P 10250 5550
-F 0 "R?" V 10330 5500 50  0000 C CNN
+F 0 "R9" V 10330 5500 50  0000 C CNN
 F 1 "500k" V 10170 5610 50  0000 C CNN
 F 2 "~" H 10250 5550 60  0000 C CNN
@@
 $EndComp
 $Comp
-L SPST SW?
+L SPST SW1
 U 1 1 561660B0
 P 8200 3300
-F 0 "SW?" H 8200 3400 70  0000 C CNN
+F 0 "SW1" H 8200 3400 70  0000 C CNN
 F 1 "SPST" H 8200 3200 70  0000 C CNN
 F 2 "~" H 8200 3300 60  0000 C CNN
@@
 $EndComp
 $Comp
-L SPST SW?
+L SPST SW2
 U 1 1 561660D3
 P 9000 3100
-F 0 "SW?" H 9000 3200 70  0000 C CNN
+F 0 "SW2" H 9000 3200 70  0000 C CNN
 F 1 "SPST" H 9000 3000 70  0000 C CNN
 F 2 "~" H 9000 3100 60  0000 C CNN
@@
 $EndComp
 $Comp
-L SPST SW?
+L SPST SW3
 U 1 1 561660D9
 P 9800 2850
-F 0 "SW?" H 9800 2950 70  0000 C CNN
+F 0 "SW3" H 9800 2950 70  0000 C CNN
 F 1 "SPST" H 9800 2750 70  0000 C CNN
 F 2 "~" H 9800 2850 60  0000 C CNN
@@
 $EndComp
 $Comp
-L SPST SW?
+L SPST SW4
 U 1 1 561660E0
 P 10600 3300
-F 0 "SW?" H 10600 3400 70  0000 C CNN
+F 0 "SW4" H 10600 3400 70  0000 C CNN
 F 1 "SPST" H 10600 3200 70  0000 C CNN
 F 2 "~" H 10600 3300 60  0000 C CNN
@@
 $EndComp
 $Comp
-L SPST SW?
+L SPST SW5
 U 1 1 561660E9
 P 11400 3100
-F 0 "SW?" H 11400 3200 70  0000 C CNN
+F 0 "SW5" H 11400 3200 70  0000 C CNN
 F 1 "SPST" H 11400 3000 70  0000 C CNN
 F 2 "~" H 11400 3100 60  0000 C CNN
@@
 $EndComp
 $Comp
-L SPST SW?
+L SPST SW6
 U 1 1 561660EF
 P 12200 2850
-F 0 "SW?" H 12200 2950 70  0000 C CNN
+F 0 "SW6" H 12200 2950 70  0000 C CNN
 F 1 "SPST" H 12200 2750 70  0000 C CNN
 F 2 "~" H 12200 2850 60  0000 C CNN
@@
 $EndComp
 $Comp
-L CP1 C?
+L CP1 C2
 U 1 1 561665DD
 P 8300 8250
-F 0 "C?" H 8350 8350 50  0000 L CNN
+F 0 "C2" H 8350 8350 50  0000 L CNN
 F 1 "100u" H 8350 8150 50  0000 L CNN
 F 2 "~" H 8300 8250 60  0000 C CNN
@@
 $EndComp
 $Comp
-L CP1 C?
+L CP1 C6
 U 1 1 56166602
 P 9500 8250
-F 0 "C?" H 9550 8350 50  0000 L CNN
+F 0 "C6" H 9550 8350 50  0000 L CNN
 F 1 "100u" H 9550 8150 50  0000 L CNN
 F 2 "~" H 9500 8250 60  0000 C CNN
@@
 $EndComp
 $Comp
-L CP1 C?
+L CP1 C4
 U 1 1 56166608
 P 8800 9550
-F 0 "C?" H 8850 9650 50  0000 L CNN
+F 0 "C4" H 8850 9650 50  0000 L CNN
 F 1 "470u" H 8850 9450 50  0000 L CNN
 F 2 "~" H 8800 9550 60  0000 C CNN
@@
 Wire Wire Line
 	9300 5950 9500 5950
-Wire Wire Line
-	14300 6050 14300 5750
 Wire Wire Line
 	8100 6150 7400 6150
@@
 	8700 3300 8700 1950
 Connection ~ 8700 1950
+Wire Wire Line
+	7900 4150 7900 4250
 $EndSCHEMATC
